File: demo/example_1.kicad_sch (KiCad schematic)
At the start: 4 parts, among them U1 24C02

Commit message: Update example project to illustrate usage of properties
Parts:
- R1: KiVar.Rule EEPROM_ADDR 0x55() *(-!) -> EEPROM_ADDR 0x55(+!)
- R2: KiVar.Rule EEPROM_ADDR 0x54() *(-!) -> EEPROM_ADDR 0x54(+!)
Changed lines of the file:
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@@
 			)
 		)
-		(property "KiVar.Rule" "EEPROM_ADDR 0x54() *(-!)"
+		(property "KiVar.Rule" "EEPROM_ADDR 0x54(+!)"
 			(at 95.25 66.0399 0)
 			(effects
@@
 			)
 		)
-		(property "KiVar.Rule" "EEPROM_ADDR 0x55() *(-!)"
+		(property "KiVar.Rule" "EEPROM_ADDR 0x55(+!)"
 			(at 95.25 55.8799 0)
 			(effects
