File: demo/example_1.kicad_sch (KiCad schematic)
At the start: 4 parts, among them U1 24C02

Commit message: For each aspect, add a "VarID" field in an essential component to create a board variant ID code
Parts:
- U1: VarID (none) -> 55; VarID.Var (none) -> 0x54(54) 0x55(55)
Changed lines of the file:
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@@
 	(title_block
 		(title "KiVar Demo")
-		(date "2024-05-29")
-		(rev "0.2.0")
+		(date "2024-07-11")
+		(rev "0.3.0")
 		(company "Author: Mark Hämmerling <dev@markh.de>")
 		(comment 1 "https://github.com/markh-de/KiVar")
@@
 			(at 119.38 60.96 0)
 			(effects
+				(font
+					(size 1.27 1.27)
+				)
+				(hide yes)
+			)
+		)
+		(property "VarID" "55"
+			(at 119.38 60.96 0)
+			(effects
+				(font
+					(size 1.27 1.27)
+				)
+				(hide yes)
+			)
+		)
+		(property "VarID.Var" "0x54(54) 0x55(55)"
+			(at 119.38 60.96 0)
+			(effects
