File: demo/kivar-demo.kicad_pcb (KiCad board)
At the start: 2 copper layers, 57 x 36 mm, 61 parts, among them U1 24C02, U2 MIC841HYC5, U3 ISL91127IR, U4 TCA9535PWR, U5 TCA9539PWR, U6 AP3032

Commit message: Make use of new 0.2.0 features in demo project, use different expression types
Parts:
- removed U5: TCA9539PWR, Package_SO:TSSOP-24_4.4x7.8mm_P0.65mm
- U3: value ISL91127IR -> ISL91127IRAZ
Connections:
- net /Example 4: IC Variant Selection/BB_FB renamed Net-(U3-FB)
- U4 pad 1: /Example 5: IC Type and Address Selection/~{INT} -> unconnected-(U4-~{INT}-Pad1)
- U4 pad 10: /Example 5: IC Type and Address Selection/P06 -> unconnected-(U4-P06-Pad10)
- U4 pad 11: /Example 5: IC Type and Address Selection/P07 -> unconnected-(U4-P07-Pad11)
- U4 pad 13: /Example 5: IC Type and Address Selection/P10 -> unconnected-(U4-P10-Pad13)
- U4 pad 14: /Example 5: IC Type and Address Selection/P11 -> unconnected-(U4-P11-Pad14)
- U4 pad 15: /Example 5: IC Type and Address Selection/P12 -> unconnected-(U4-P12-Pad15)
- U4 pad 16: /Example 5: IC Type and Address Selection/P13 -> unconnected-(U4-P13-Pad16)
- U4 pad 17: /Example 5: IC Type and Address Selection/P14 -> unconnected-(U4-P14-Pad17)
- U4 pad 18: /Example 5: IC Type and Address Selection/P15 -> unconnected-(U4-P15-Pad18)
- U4 pad 19: /Example 5: IC Type and Address Selection/P16 -> unconnected-(U4-P16-Pad19)
- U4 pad 20: /Example 5: IC Type and Address Selection/P17 -> unconnected-(U4-P17-Pad20)
- U4 pad 4: /Example 5: IC Type and Address Selection/P00 -> unconnected-(U4-P00-Pad4)
- U4 pad 5: /Example 5: IC Type and Address Selection/P01 -> unconnected-(U4-P01-Pad5)
- U4 pad 6: /Example 5: IC Type and Address Selection/P02 -> unconnected-(U4-P02-Pad6)
- U4 pad 7: /Example 5: IC Type and Address Selection/P03 -> unconnected-(U4-P03-Pad7)
- U4 pad 8: /Example 5: IC Type and Address Selection/P04 -> unconnected-(U4-P04-Pad8)
- U4 pad 9: /Example 5: IC Type and Address Selection/P05 -> unconnected-(U4-P05-Pad9)
