File: demo/example_2.kicad_sch (KiCad schematic)
At the start: 12 parts

Commit message: For each aspect, add a "VarID" field in an essential component to create a board variant ID code
Parts:
- R9: VarID (none) -> E; VarID.Var (none) -> SD(S) EMMC(E) NAND(N) JP(J)
Changed lines of the file:
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@@
 	(title_block
 		(title "KiVar Demo")
-		(date "2024-05-29")
-		(rev "0.2.0")
+		(date "2024-07-11")
+		(rev "0.3.0")
 		(company "Author: Mark Hämmerling <dev@markh.de>")
 		(comment 1 "https://github.com/markh-de/KiVar")
@@
 			)
 		)
+		(property "VarID" "E"
+			(at 139.065 85.09 0)
+			(effects
+				(font
+					(size 1.27 1.27)
+				)
+				(hide yes)
+			)
+		)
+		(property "VarID.Var" "SD(S) EMMC(E) NAND(N) JP(J)"
+			(at 139.065 85.09 0)
+			(effects
+				(font
+					(size 1.27 1.27)
+				)
+				(hide yes)
+			)
+		)
