File: demo/example_2.kicad_sch (KiCad schematic)
At the start: 12 parts

Commit message: Demo: Switch state to specific variant
Parts:
- R10: now fitted; now in the parts list
- R11: now not fitted; now left out of the parts list
- R9: ChoiceText SoM eMMC -> SoM NAND; VarID E -> N; now not fitted; now left out of the parts list
Changed lines of the file:
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@@
 		(unit 1)
 		(exclude_from_sim no)
-		(in_bom yes)
-		(on_board yes)
-		(dnp no)
+		(in_bom no)
+		(on_board yes)
+		(dnp yes)
 		(property "Reference" "R9"
 			(at 140.97 82.5499 0)
@@
 			)
 		)
-		(property "ChoiceText" "SoM eMMC"
+		(property "ChoiceText" "SoM NAND"
 			(at 139.065 85.09 0)
 			(effects
@@
 			)
 		)
-		(property "VarID" "E"
+		(property "VarID" "N"
 			(at 139.065 85.09 0)
 			(effects
@@
 		(unit 1)
 		(exclude_from_sim no)
-		(in_bom no)
-		(on_board yes)
-		(dnp yes)
+		(in_bom yes)
+		(on_board yes)
+		(dnp no)
 		(fields_autoplaced yes)
 		(property "Reference" "R10"
@@
 		(unit 1)
 		(exclude_from_sim no)
-		(in_bom yes)
-		(on_board yes)
-		(dnp no)
+		(in_bom no)
+		(on_board yes)
+		(dnp yes)
 		(fields_autoplaced yes)
 		(property "Reference" "R11"
