File: demo/example_3.kicad_sch (KiCad schematic)
At the start: 6 parts, among them U2 MIC841HYC5

Commit message: For each aspect, add a "VarID" field in an essential component to create a board variant ID code
Parts:
- R12: VarID (none) -> 3; VarID.Var (none) -> '2.41V/3.40V'(2) '3.15V/3.57V'(3)
Changed lines of the file:
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@@
 	(title_block
 		(title "KiVar Demo")
-		(date "2024-05-29")
-		(rev "0.2.0")
+		(date "2024-07-11")
+		(rev "0.3.0")
 		(company "Author: Mark Hämmerling <dev@markh.de>")
 		(comment 1 "https://github.com/markh-de/KiVar")
@@
 			)
 		)
+		(property "VarID" "3"
+			(at 108.585 50.8 0)
+			(effects
+				(font
+					(size 1.27 1.27)
+				)
+				(hide yes)
+			)
+		)
+		(property "VarID.Var" "'2.41V/3.40V'(2) '3.15V/3.57V'(3)"
+			(at 108.585 50.8 0)
+			(effects
+				(font
+					(size 1.27 1.27)
+				)
+				(hide yes)
+			)
+		)

Commit message: Clean up demo project fields a bit
Other:
- note removed: "TODO: Update component values according to real project."
Changed lines of the file:
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@@
-		)
-	)
-	(text "TODO: Update component values according to real project."
-		(exclude_from_sim no)
-		(at 105.41 34.29 0)
-		(effects
-			(font
-				(size 1.27 1.27)
-			)
 		)
 	)
@@
 			)
 		)
+		(property "Var.Aspect" "UVLO_LO/HI"
+			(at 108.585 68.58 0)
+			(effects
+				(font
+					(size 1.27 1.27)
+				)
+				(hide yes)
+			)
+		)
 		(property "Var" "'2.41V/3.40V'(309kΩ) '3.15V/3.57V'(100kΩ)"
 			(at 106.68 71.1199 0)
@@
 				)
 				(justify right)
-			)
-		)
-		(property "Var.Aspect" "UVLO_LO/HI"
-			(at 108.585 68.58 0)
-			(effects
-				(font
-					(size 1.27 1.27)
-				)
-				(hide yes)
 			)
 		)
@@
 				)
 				(hide yes)
-			)
-		)
-		(property "Var" "'2.41V/3.40V'(0Ω) '3.15V/3.57V'(309kΩ)"
-			(at 106.68 53.3399 0)
-			(effects
-				(font
-					(size 1.27 1.27)
-					(italic yes)
-				)
-				(justify left)
 			)
 		)
@@
 			)
 		)
+		(property "Var" "'2.41V/3.40V'(0Ω) '3.15V/3.57V'(309kΩ)"
+			(at 106.68 53.3399 0)
+			(effects
+				(font
+					(size 1.27 1.27)
+					(italic yes)
+				)
+				(justify left)
+			)
+		)
 		(property "VarID" "3"
 			(at 108.585 50.8 0)
@@
 			)
 		)
+		(property "Var.Aspect" "UVLO_LO/HI"
+			(at 108.585 77.47 0)
+			(effects
+				(font
+					(size 1.27 1.27)
+				)
+				(hide yes)
+			)
+		)
 		(property "Var" "*(750kΩ)"
 			(at 106.68 80.0099 0)
@@
 				)
 				(justify left)
-			)
-		)
-		(property "Var.Aspect" "UVLO_LO/HI"
-			(at 108.585 77.47 0)
-			(effects
-				(font
-					(size 1.27 1.27)
-				)
-				(hide yes)
 			)
 		)
@@
 			)
 		)
+		(property "Var.Aspect" "UVLO_LO/HI"
+			(at 108.585 59.69 0)
+			(effects
+				(font
+					(size 1.27 1.27)
+				)
+				(hide yes)
+			)
+		)
 		(property "Var" "*(1MΩ)"
 			(at 106.68 62.2299 0)
@@
 			)
 		)
-		(property "Var.Aspect" "UVLO_LO/HI"
-			(at 108.585 59.69 0)
-			(effects
-				(font
-					(size 1.27 1.27)
-				)
-				(hide yes)
-			)
-		)
