File: demo/example_4.kicad_sch (KiCad schematic)
At the start: 10 parts, among them U3 ISL91127IRAZ

Commit message: For each aspect, add a "VarID" field in an essential component to create a board variant ID code
Parts:
- U3: VarID (none) -> A; VarID.Var (none) -> IRAZ(A) IRNZ(N)
Changed lines of the file:
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@@
 	(title_block
 		(title "KiVar Demo")
-		(date "2024-05-29")
-		(rev "0.2.0")
+		(date "2024-07-11")
+		(rev "0.3.0")
 		(company "Author: Mark Hämmerling <dev@markh.de>")
 		(comment 1 "https://github.com/markh-de/KiVar")
@@
 				(hide yes)
 			)
+		)
+		(property "VarID" "A"
+			(at 121.92 104.14 0)
+			(effects
+				(font
+					(size 1.27 1.27)
+				)
+				(hide yes)
+			)
+		)
+		(property "VarID.Var" "IRAZ(A) IRNZ(N)"
+			(at 121.92 104.14 0)
+			(effects
+				(font
+					(size 1.27 1.27)
+				)
+				(hide yes)
+			)
