File: demo/example_4.kicad_sch (KiCad schematic)
At the start: 10 parts, among them U3 ISL91127IRAZ

Commit message: Demo: Switch state to specific variant
Parts:
- C5, C6, R17: now not fitted; now left out of the parts list
- R16: value 1MΩ -> 0Ω
- U3: value ISL91127IRAZ -> ISL91127IRNZ; Info Adjustable -> Fixed; MPN ISL91127IRAZ-T7A -> ISL91127IRNZ-T7A; VarID A -> N
Changed lines of the file:
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@@
 			)
 		)
-		(property "Value" "1MΩ"
+		(property "Value" "0Ω"
 			(at 176.53 101.5999 0)
 			(effects
@@
 			)
 		)
-		(property "Value" "ISL91127IRAZ"
+		(property "Value" "ISL91127IRNZ"
 			(at 127.9241 87.63 0)
 			(effects
@@
 			)
 		)
-		(property "MPN" "ISL91127IRAZ-T7A"
+		(property "MPN" "ISL91127IRNZ-T7A"
 			(at 121.92 104.14 0)
 			(effects
@@
 			)
 		)
-		(property "Info" "Adjustable"
+		(property "Info" "Fixed"
 			(at 127.9241 90.17 0)
 			(effects
@@
 			)
 		)
-		(property "VarID" "A"
+		(property "VarID" "N"
 			(at 121.92 104.14 0)
 			(effects
@@
 		(unit 1)
 		(exclude_from_sim no)
-		(in_bom yes)
-		(on_board yes)
-		(dnp no)
+		(in_bom no)
+		(on_board yes)
+		(dnp yes)
 		(fields_autoplaced yes)
 		(property "Reference" "C6"
@@
 		(unit 1)
 		(exclude_from_sim no)
-		(in_bom yes)
-		(on_board yes)
-		(dnp no)
+		(in_bom no)
+		(on_board yes)
+		(dnp yes)
 		(fields_autoplaced yes)
 		(property "Reference" "R17"
@@
 		(unit 1)
 		(exclude_from_sim no)
-		(in_bom yes)
-		(on_board yes)
-		(dnp no)
+		(in_bom no)
+		(on_board yes)
+		(dnp yes)
 		(fields_autoplaced yes)
 		(property "Reference" "C5"
