File: demo/example_5.kicad_sch (KiCad schematic)
At the start: 5 parts, among them U4 TCA9535PWR

Commit message: For each aspect, add a "VarID" field in an essential component to create a board variant ID code
Parts:
- U4: VarID (none) -> 24; VarID.Var (none) -> 9535/0x20(20) 9535/0x24(24) 9539/0x74(74)
Changed lines of the file:
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@@
 	(title_block
 		(title "KiVar Demo")
-		(date "2024-05-29")
-		(rev "0.2.0")
+		(date "2024-07-11")
+		(rev "0.3.0")
 		(company "Author: Mark Hämmerling <dev@markh.de>")
 		(comment 1 "https://github.com/markh-de/KiVar")
@@
 			(at 170.18 100.33 0)
 			(effects
+				(font
+					(size 1.27 1.27)
+				)
+				(hide yes)
+			)
+		)
+		(property "VarID" "24"
+			(at 170.18 100.33 0)
+			(effects
+				(font
+					(size 1.27 1.27)
+				)
+				(hide yes)
+			)
+		)
+		(property "VarID.Var" "9535/0x20(20) 9535/0x24(24) 9539/0x74(74)"
+			(at 170.18 100.33 0)
+			(effects

Commit message: Demo: Switch 3D models
Parts:
- U4: Var(*) (none) -> +m1-m2; Var(9539/0x74) (none) -> -m1+m2
Changed lines of the file:
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@@
+			)
+		)
+		(property "Var(*)" "+m1-m2"
+			(at 170.18 100.33 0)
+			(effects
+				(font
+					(size 1.27 1.27)
+				)
+				(hide yes)
+			)
+		)
+		(property "Var(9539/0x74)" "-m1+m2"
+			(at 170.18 100.33 0)
+			(effects
+				(font
+					(size 1.27 1.27)
+				)
+				(hide yes)
 			)
 		)

Commit message: Clean up demo project fields a bit
Parts:
- U4: Var *(TCA9535PWR) 9539/0x74(TCA9539PWR) -> *(TCA9535PWR +m1-m2) 9539/0x74(TCA9539PWR -m1+m2); Var(*) +m1-m2 -> (none); Var(9539/0x74) -m1+m2 -> (none)
Changed lines of the file:
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@@
 			)
 		)
-		(property "Var" "*(TCA9535PWR) 9539/0x74(TCA9539PWR)"
+		(property "Var" "*(TCA9535PWR +m1-m2) 9539/0x74(TCA9539PWR -m1+m2)"
 			(at 172.3741 74.93 0)
 			(effects
@@
 			)
 		)
-		(property "Var(*)" "+m1-m2"
-			(at 170.18 100.33 0)
-			(effects
-				(font
-					(size 1.27 1.27)
-				)
-				(hide yes)
-			)
-		)
-		(property "Var(9539/0x74)" "-m1+m2"
+		(property "Datasheet.Var(*)" "http://www.ti.com/lit/ds/symlink/tca9535.pdf"
 			(at 170.18 100.33 0)
 			(effects
@@
 			)
 		)
-		(property "Datasheet.Var(*)" "http://www.ti.com/lit/ds/symlink/tca9535.pdf"
+		(property "MPN.Var(*)" "TCA9535PWR"
 			(at 170.18 100.33 0)
 			(effects
@@
 			(at 170.18 100.33 0)
 			(effects
-				(font
-					(size 1.27 1.27)
-				)
-				(hide yes)
-			)
-		)
-		(property "MPN.Var(*)" "TCA9535PWR"
-			(at 170.18 100.33 0)
-			(effects
