File: demo/example_5.kicad_sch (KiCad schematic)
At the start: 5 parts, among them U4 TCA9535PWR

Commit message: Demo project: Use Stand-In choices where useful
Parts:
- U4: Var *(TCA9535PWR +m1-m2) 9539/0x74(TCA9539PWR -m1+m2) -> ?(TCA9535PWR +m1) 9539/0x74(TCA9539PWR +m2)
Changed lines of the file:
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@@
 	(title_block
 		(title "KiVar Demo")
-		(date "2024-07-21")
+		(date "2024-08-17")
 		(rev "0.4.0")
 		(company "Author: Mark Hämmerling <dev@markh.de>")
@@
 	(rectangle
 		(start 86.36 59.69)
-		(end 215.9 137.16)
+		(end 227.33 137.16)
 		(stroke
 			(width 0.254)
@@
 			)
 		)
-		(property "Var" "*(TCA9535PWR +m1-m2) 9539/0x74(TCA9539PWR -m1+m2)"
+		(property "Var" "?(TCA9535PWR +m1) 9539/0x74(TCA9539PWR +m2)"
 			(at 172.3741 74.93 0)
 			(effects
