File: demo/example_6.kicad_sch (KiCad schematic)
At the start: 23 parts, among them U6 AP3032

Commit message: Fix demo project for 0.4.0 re-release
Parts:
- renumbered U6 to U5
Changed lines of the file:
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@@
 	(title_block
 		(title "KiVar Demo")
-		(date "2024-09-14")
+		(date "2024-09-16")
 		(rev "0.4.0")
 		(company "Author: Mark Hämmerling <dev@markh.de>")
@@
 		(dnp no)
 		(fields_autoplaced yes)
-		(property "Reference" "U6"
+		(property "Reference" "U5"
 			(at 104.14 49.53 0)
 			(effects
@@
 			(project "kivar-demo"
 				(path "/cd745a5c-45fb-4106-85c8-c86c130b6ee7/efd04459-986c-49c2-bdc3-96a700b4a724"
-					(reference "U6")
+					(reference "U5")
 					(unit 1)
 				)
