File: demo/example_7.kicad_sch (KiCad schematic)
At the start: 6 parts, among them U5 LDO

Commit message: Fix demo project for 0.4.0 re-release
Parts:
- R34: VarID.Var 1.2V(12) 1.8V(18) 3.3V(33) -> 1.2V(12) 1.8V(18) 2.5V(25) 3.3V(33)
- renumbered U5 to U6
Changed lines of the file:
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@@
 	(title_block
 		(title "KiVar Demo")
-		(date "2024-09-14")
+		(date "2024-09-16")
 		(rev "0.4.0")
 		(company "Author: Mark Hämmerling <dev@markh.de>")
@@
 			)
 		)
-		(property "VarID.Var" "1.2V(12) 1.8V(18) 3.3V(33)"
+		(property "VarID.Var" "1.2V(12) 1.8V(18) 2.5V(25) 3.3V(33)"
 			(at 104.14 57.15 0)
 			(effects
@@
 		(on_board yes)
 		(dnp no)
-		(property "Reference" "U5"
+		(property "Reference" "U6"
 			(at 83.82 46.99 0)
 			(effects
@@
 			(project "kivar-demo"
 				(path "/cd745a5c-45fb-4106-85c8-c86c130b6ee7/6cc89fe7-613b-41f0-9c47-85b72f1b3014"
-					(reference "U5")
+					(reference "U6")
 					(unit 1)
 				)
